File: PCB/fp.kicad_sch (KiCad schematic)
At the start: 29 parts, among them J1 Line Out

Commit message: Update to Kicad 10
Changes: Moved some traces around to allow more ground fill
Parts:
- S1: value AR Mod -> AR Mod
- S3, S9: value ~ -> (none)
- S6: value VCF Mod -> VCF Mod
